File: KiCad/ESP32_blAudio_portable.kicad_sch (KiCad schematic)
At the start: 33 parts, among them J1 Conn_01x15_Male, J2 Conn_01x15_Male, J3 Conn_01x02_Male, Q1 Q_NMOS_DGS, Q2 Q_PMOS_DGS, SW1 SW_Push, SW2 SW_Push, SW3 SW_Push, SW4 RotaryEncoder_Switch, SW5 SW_Push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

Commit message: -associated footprints to more specific components -added manufacturer and part series info to more specific components
Parts:
- C1, C2: value C -> 1u
- RV1: value 100k_lin -> PT01; footprint (none) -> Potentiometer_THT:Potentiometer_Bourns_PTV09A-1_Single_Vertical; MFG (none) -> CUI Devices
- SW1, SW2, SW3, SW5: value SW_Push -> TS02; MFG (none) -> CUI Devices
- SW4: value RotaryEncoder_Switch -> PEC12R; footprint (none) -> Rotary_Encoder:RotaryEncoder_Alps_EC11E-Switch_Vertical_H20mm; MFG (none) -> Bourns Inc.
Other:
- sheet AK5720 ports: added 3-5_SW; removed none

Commit message: -layout work
Parts:
- removed R10, R8, R9: 22R, Resistor_SMD:R_0603_1608Metric, symbol Device:R
Connections:
- net GND: now also J1.14 (Pin_14), J2.14 (Pin_14)
- net LRCK2: now also J2.2 (Pin_2)
- net MCLK: now also J2.3 (Pin_3)
- net SCK2: now also J2.4 (Pin_4)
- net SDI2: now also J2.1 (Pin_1)
- net ~{PDN}: now also J2.5 (Pin_5)

Commit message: -layout work
Parts:
- added C25, C26: 1u, Capacitor_SMD:C_0603_1608Metric, symbol Device:C
- added U7: NCP1117-3.3_SOT223, Package_TO_SOT_SMD:SOT-223-3_TabPin2, symbol Regulator_Linear:NCP1117-3.3_SOT223
- Q1: value Q_NMOS_DGS -> 2N7002; footprint (none) -> Package_TO_SOT_SMD:SOT-323_SC-70; symbol Device:Q_NMOS_DGS -> Device:Q_NMOS_GSD; MFG (none) -> Nexperia USA Inc.; MFG# (none) -> 2N7002PW,115
- Q2: footprint (none) -> Package_TO_SOT_SMD:SOT-23-6; MFG (none) -> Panjit International Inc.; MFG# (none) -> PJS6403_S1_00001
Connections:
- net +3V3: now also J1.1 (Pin_1), J2.15 (Pin_15), C26.1, U7.2 (VO)
- net +VDC: now also C25.1, U7.3 (VI)
- net ANA_VOL: now also J1.9 (Pin_9)
- net BTTN1: now also J2.11 (Pin_11)
- net BTTN2: now also J2.12 (Pin_12)
- net BTTN3: now also J2.13 (Pin_13)
- net ENC_A: now also J1.7 (Pin_7)
- net ENC_B: now also J1.8 (Pin_8)
- net ENC_SW: now also J1.6 (Pin_6)
- net EN_5V: now also J1.3 (Pin_3)
- net GND: now also Q1.2 (S), C25.2, C26.2, U7.1 (GND); no longer Q1.3 (S)
- net LED1: now also J2.9 (Pin_9)
- net LED2: now also J2.10 (Pin_10)
- net LRCK1: now also J2.6 (Pin_6)
- net PWR_ON: now also J1.2 (Pin_2)
- net SCK1: now also J2.7 (Pin_7)
- net SCL: now also J1.4 (Pin_4)
- net SDA: now also J1.5 (Pin_5)
- net SDI1: now also J2.8 (Pin_8)
- net at R11.2, R13.1: now also Q1.1 (G); no longer Q1.2 (G)
- net at Q2.2 (G), R12.2, SW5.2: now also Q1.3 (D); no longer Q1.1 (D)
Other:
- moved on the sheet: JP1, Q1, Q2, R11, R12, R13, SW5

Commit message: -layout largely finished, some finishing touches needed
Connections:
- net 3-5_SW: now also J1.13 (Pin_13)
Changed lines of the file:
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@@
+    (stroke (width 0) (type default) (color 0 0 0 0))
+  )
+  (wire (pts (xy 95.25 60.96) (xy 97.79 60.96))
     (stroke (width 0) (type default) (color 0 0 0 0))
   )
@@
     (effects (font (size 1.27 1.27)) (justify left bottom))
   )
+  (label "3-5_SW" (at 95.25 60.96 180)
+    (effects (font (size 1.27 1.27)) (justify right bottom))
+  )
   (label "BTTN2" (at 137.16 58.42 0)

Commit message: -First board version ready to order
Parts:
- Q2: value Q_PMOS_DGS -> PJS6403
Changed lines of the file:
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@@
     (in_bom yes) (on_board yes) (fields_autoplaced)
     (property "Reference" "Q2" (id 0) (at 227.33 113.03 90))
-    (property "Value" "Q_PMOS_DGS" (id 1) (at 227.33 115.57 90))
+    (property "Value" "PJS6403" (id 1) (at 227.33 115.57 90))
     (property "Footprint" "Package_TO_SOT_SMD:SOT-23-6" (id 2) (at 229.87 118.11 0)
       (effects (font (size 1.27 1.27)) hide)
@@
     )
     (path "/7daad98a-6199-4c54-9ede-821fd2d474ad"
-      (reference "Q2") (unit 1) (value "Q_PMOS_DGS") (footprint "Package_TO_SOT_SMD:SOT-23-6")
+      (reference "Q2") (unit 1) (value "PJS6403") (footprint "Package_TO_SOT_SMD:SOT-23-6")
     )
     (path "/75a8b4cf-be6c-4d23-8740-2e62cd0245ef/9e63908d-f4de-4538-8c1e-c9fc793744b4"

Commit message: -boards on hand atm, assembling first board and finalizing used component values
Parts:
- R1, R2, R5: value 10k -> NP
- R6, R7: value 10k -> 2k2
Other:
- note added: "Changes to next version: -series resistor to ESP32's EN line -(low) optimize pot and encoder footprints"
Changed lines of the file:
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@@
     (effects (font (size 1.58 1.58)) (justify right bottom))
+  )
+  (text "Changes to next version:\n-series resistor to ESP32's EN line\n-(low) optimize pot and encoder footprints"
+    (at 96.52 -20.32 0)
+    (effects (font (size 1.27 1.27)) (justify left bottom))
   )
   (text "power-up\nbutton" (at 245.11 148.59 0)
@@
       (effects (font (size 1.27 1.27)) (justify right))
     )
-    (property "Value" "10k" (id 1) (at 88.9 181.6099 0)
+    (property "Value" "2k2" (id 1) (at 88.9 181.6099 0)
       (effects (font (size 1.27 1.27)) (justify right))
     )
@@
       (effects (font (size 1.27 1.27)) (justify right))
     )
-    (property "Value" "10k" (id 1) (at 128.27 163.8299 0)
+    (property "Value" "2k2" (id 1) (at 128.27 163.8299 0)
       (effects (font (size 1.27 1.27)) (justify right))
     )
@@
       (effects (font (size 1.27 1.27)) (justify right))
     )
-    (property "Value" "10k" (id 1) (at 25.4 165.0999 0)
+    (property "Value" "NP" (id 1) (at 25.4 165.0999 0)
       (effects (font (size 1.27 1.27)) (justify right))
     )
@@
       (effects (font (size 1.27 1.27)) (justify right))
     )
-    (property "Value" "10k" (id 1) (at 53.34 165.0999 0)
+    (property "Value" "NP" (id 1) (at 53.34 165.0999 0)
       (effects (font (size 1.27 1.27)) (justify right))
     )
@@
       (effects (font (size 1.27 1.27)) (justify right))
     )
-    (property "Value" "10k" (id 1) (at 39.37 165.0999 0)
+    (property "Value" "NP" (id 1) (at 39.37 165.0999 0)
       (effects (font (size 1.27 1.27)) (justify right))
     )
@@
     )
     (path "/fe9cb004-3747-4931-bcd5-b57852eb813d/1de3fe4d-6b8d-4612-8808-f29a2b0fe5ca"
-      (reference "C15") (unit 1) (value "10µ") (footprint "Capacitor_SMD:C_0603_1608Metric")
+      (reference "C15") (unit 1) (value "1u") (footprint "Capacitor_SMD:C_0603_1608Metric")
     )
     (path "/fe9cb004-3747-4931-bcd5-b57852eb813d/d5200166-3d95-4e0a-98cb-787606a3056b"
-      (reference "C16") (unit 1) (value "1µ") (footprint "Capacitor_SMD:C_0603_1608Metric")
+      (reference "C16") (unit 1) (value "1u") (footprint "Capacitor_SMD:C_0603_1608Metric")
     )
     (path "/fe9cb004-3747-4931-bcd5-b57852eb813d/df2ba706-5f04-4899-bbe5-56b5b2ba018b"
-      (reference "C17") (unit 1) (value "10µ") (footprint "Capacitor_SMD:C_0603_1608Metric")
+      (reference "C17") (unit 1) (value "1u") (footprint "Capacitor_SMD:C_0603_1608Metric")
     )
     (path "/fe9cb004-3747-4931-bcd5-b57852eb813d/3cadabd0-3a7e-4ef6-a636-c508c5af13f4"
-      (reference "C18") (unit 1) (value "1µ") (footprint "Capacitor_SMD:C_0603_1608Metric")
+      (reference "C18") (unit 1) (value "1u") (footprint "Capacitor_SMD:C_0603_1608Metric")
     )
     (path "/fe9cb004-3747-4931-bcd5-b57852eb813d/6551e401-e320-4e15-8a96-847c2ff286e2"
-      (reference "C19") (unit 1) (value "1µ") (footprint "Capacitor_SMD:C_0603_1608Metric")
+      (reference "C19") (unit 1) (value "1u") (footprint "Capacitor_SMD:C_0603_1608Metric")
     )
     (path "/fe9cb004-3747-4931-bcd5-b57852eb813d/fc6022fe-f428-4c00-b3ee-86b0895d6e55"
-      (reference "C20") (unit 1) (value "220n") (footprint "Capacitor_SMD:C_0603_1608Metric")
+      (reference "C20") (unit 1) (value "1u") (footprint "Capacitor_SMD:C_0603_1608Metric")
     )
     (path "/fe9cb004-3747-4931-bcd5-b57852eb813d/703b90db-3767-4042-9985-be5b95a6b104"
-      (reference "C21") (unit 1) (value "1µ") (footprint "Capacitor_SMD:C_0603_1608Metric")
+      (reference "C21") (unit 1) (value "1u") (footprint "Capacitor_SMD:C_0603_1608Metric")
     )
     (path "/75a8b4cf-be6c-4d23-8740-2e62cd0245ef/e38bc2e8-6ea3-4667-9fea-8bd68c0690a8"
@@
     )
     (path "/9202587a-b087-4076-8b92-570a03f50eaf"
-      (reference "R1") (unit 1) (value "10k") (footprint "Resistor_SMD:R_0603_1608Metric")
+      (reference "R1") (unit 1) (value "NP") (footprint "Resistor_SMD:R_0603_1608Metric")
     )
     (path "/f1bad60c-0405-43c1-a1cb-7d64ac9c33ee"
-      (reference "R2") (unit 1) (value "10k") (footprint "Resistor_SMD:R_0603_1608Metric")
+      (reference "R2") (unit 1) (value "NP") (footprint "Resistor_SMD:R_0603_1608Metric")
     )
     (path "/30b45333-af19-4d55-a3b8-c3e5383806e0"
@@
     )
     (path "/c70720be-76b3-4bb2-b393-f348d7f1d2c1"
-      (reference "R5") (unit 1) (value "10k") (footprint "Resistor_SMD:R_0603_1608Metric")
+      (reference "R5") (unit 1) (value "NP") (footprint "Resistor_SMD:R_0603_1608Metric")
     )
     (path "/0807fc2c-4a20-4527-be5c-b89cd35731b1"
-      (reference "R6") (unit 1) (value "10k") (footprint "Resistor_SMD:R_0603_1608Metric")
+      (reference "R6") (unit 1) (value "2k2") (footprint "Resistor_SMD:R_0603_1608Metric")
     )
     (path "/8d900974-7a7b-4b9a-a18a-6e547d74dd75"
-      (reference "R7") (unit 1) (value "10k") (footprint "Resistor_SMD:R_0603_1608Metric")
+      (reference "R7") (unit 1) (value "2k2") (footprint "Resistor_SMD:R_0603_1608Metric")
     )
     (path "/539e998b-d3fa-4051-8795-c2eb17e77d37"
@@
     )
     (path "/fe9cb004-3747-4931-bcd5-b57852eb813d/6182ab49-5007-4619-a7fc-fabbee725405"
-      (reference "R32") (unit 1) (value "R") (footprint "Resistor_SMD:R_0603_1608Metric")
+      (reference "R32") (unit 1) (value "22R") (footprint "Resistor_SMD:R_0603_1608Metric")
     )
     (path "/fe9cb004-3747-4931-bcd5-b57852eb813d/b18f2a0f-c895-491a-b769-01221034684f"
-      (reference "R33") (unit 1) (value "R") (footprint "Resistor_SMD:R_0603_1608Metric")
+      (reference "R33") (unit 1) (value "0R") (footprint "Resistor_SMD:R_0603_1608Metric")
     )
     (path "/fe9cb004-3747-4931-bcd5-b57852eb813d/f02757fa-e696-4159-bd71-faa2ee166929"
-      (reference "R34") (unit 1) (value "R") (footprint "Resistor_SMD:R_0603_1608Metric")
+      (reference "R34") (unit 1) (value "NP") (footprint "Resistor_SMD:R_0603_1608Metric")
     )
     (path "/fe9cb004-3747-4931-bcd5-b57852eb813d/c84c54d0-c25c-4939-93fa-21b60cb08f98"
-      (reference "R35") (unit 1) (value "R") (footprint "Resistor_SMD:R_0603_1608Metric")
+      (reference "R35") (unit 1) (value "0R") (footprint "Resistor_SMD:R_0603_1608Metric")
     )
     (path "/fe9cb004-3747-4931-bcd5-b57852eb813d/c773e71b-79df-4f6c-ad3a-c20dcb06f5cc"
-      (reference "R36") (unit 1) (value "R") (footprint "Resistor_SMD:R_0603_1608Metric")
+      (reference "R36") (unit 1) (value "NP") (footprint "Resistor_SMD:R_0603_1608Metric")
     )
     (path "/fe9cb004-3747-4931-bcd5-b57852eb813d/3aab61b9-f5d7-4ee8-8568-52e2fa902f4f"
-      (reference "R37") (unit 1) (value "R") (footprint "Resistor_SMD:R_0603_1608Metric")
+      (reference "R37") (unit 1) (value "NP") (footprint "Resistor_SMD:R_0603_1608Metric")
     )
     (path "/fe9cb004-3747-4931-bcd5-b57852eb813d/306fae1a-e3b0-46b5-812e-cc0049e34a98"
-      (reference "R38") (unit 1) (value "R") (footprint "Resistor_SMD:R_0603_1608Metric")
+      (reference "R38") (unit 1) (value "0R") (footprint "Resistor_SMD:R_0603_1608Metric")
     )
     (path "/fe9cb004-3747-4931-bcd5-b57852eb813d/9fe1240e-ff8b-44d1-8305-09faa9aefc2b"
-      (reference "R39") (unit 1) (value "R") (footprint "Resistor_SMD:R_0603_1608Metric")
+      (reference "R39") (unit 1) (value "NP") (footprint "Resistor_SMD:R_0603_1608Metric")
     )
     (path "/fe9cb004-3747-4931-bcd5-b57852eb813d/14284b42-0f5f-40c0-881d-dd2646def4ea"
-      (reference "R40") (unit 1) (value "R") (footprint "Resistor_SMD:R_0603_1608Metric")
+      (reference "R40") (unit 1) (value "0R") (footprint "Resistor_SMD:R_0603_1608Metric")
     )
     (path "/75a8b4cf-be6c-4d23-8740-2e62cd0245ef/0cc04681-8c7b-4dee-9abc-fef5528f8ddb"

Commit message: -More HW updates and corrections -basic FW
Other:
- note added: "Changes to next version: -series resistor to ESP32's EN line -(low) optimize pot and encoder footprints -GPIOs 36, 39, 34 and 35 are INPUT ONLY"
- note removed: "Changes to next version: -series resistor to ESP32's EN line -(low) optimize pot and encoder footprints"
Changed lines of the file:
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@@
     (effects (font (size 1.58 1.58)) (justify right bottom))
   )
-  (text "Changes to next version:\n-series resistor to ESP32's EN line\n-(low) optimize pot and encoder footprints"
-    (at 96.52 -20.32 0)
-    (effects (font (size 1.27 1.27)) (justify left bottom))
+  (text "Changes to next version:\n-series resistor to ESP32's EN line\n-(low) optimize pot and encoder footprints\n-GPIOs 36, 39, 34 and 35 are INPUT ONLY"
+    (at 96.52 7.62 0)
+    (effects (font (size 2.54 2.54)) (justify left bottom))
   )
   (text "power-up\nbutton" (at 245.11 148.59 0)

Commit message: -updated schematic component values, updated schematic PDF -added simple bass and treble control for the TF9879 amp
Parts:
- R14, R15: value 10k -> 4k7
Changed lines of the file:
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@@
   )
   (text "Changes to next version:\n-series resistor to ESP32's EN line\n-(low) optimize pot and encoder footprints\n-GPIOs 36, 39, 34 and 35 are INPUT ONLY"
-    (at 96.52 7.62 0)
-    (effects (font (size 2.54 2.54)) (justify left bottom))
+    (at 109.22 109.22 0)
+    (effects (font (size 1.27 1.27)) (justify left bottom))
   )
   (text "power-up\nbutton" (at 245.11 148.59 0)
@@
       (effects (font (size 1.27 1.27)) (justify left))
     )
-    (property "Value" "10k" (id 1) (at 237.49 30.4799 0)
+    (property "Value" "4k7" (id 1) (at 237.49 30.4799 0)
       (effects (font (size 1.27 1.27)) (justify left))
     )
@@
       (effects (font (size 1.27 1.27)) (justify left))
     )
-    (property "Value" "10k" (id 1) (at 229.87 30.4799 0)
+    (property "Value" "4k7" (id 1) (at 229.87 30.4799 0)
       (effects (font (size 1.27 1.27)) (justify left))
     )
@@
     )
     (path "/6785bf95-93a5-45b5-a636-e7169bb3f708/afc7d43b-9f6f-4039-a896-6801bce38cb5"
-      (reference "C3") (unit 1) (value "100n") (footprint "Capacitor_SMD:C_0603_1608Metric")
+      (reference "C3") (unit 1) (value "1u") (footprint "Capacitor_SMD:C_0603_1608Metric")
     )
     (path "/6785bf95-93a5-45b5-a636-e7169bb3f708/70b2bcc7-30d0-4bb0-9597-39ba997d7a25"
@@
     )
     (path "/6785bf95-93a5-45b5-a636-e7169bb3f708/ea77193e-3f9c-4a16-9af4-44155de6e2bb"
-      (reference "C6") (unit 1) (value "100n") (footprint "Capacitor_SMD:C_0603_1608Metric")
+      (reference "C6") (unit 1) (value "1u") (footprint "Capacitor_SMD:C_0603_1608Metric")
     )
     (path "/6785bf95-93a5-45b5-a636-e7169bb3f708/a678b93c-ab66-4100-8ef3-b5ea0826667d"
-      (reference "C7") (unit 1) (value "100n") (footprint "Capacitor_SMD:C_0603_1608Metric")
+      (reference "C7") (unit 1) (value "1n") (footprint "Capacitor_SMD:C_0603_1608Metric")
     )
     (path "/6785bf95-93a5-45b5-a636-e7169bb3f708/f9bfe2eb-93b6-4c17-a75d-9f3361e33679"
-      (reference "C8") (unit 1) (value "100n") (footprint "Capacitor_SMD:C_0603_1608Metric")
+      (reference "C8") (unit 1) (value "1n") (footprint "Capacitor_SMD:C_0603_1608Metric")
     )
     (path "/dbae959f-bfa2-4953-9b3f-f4525f8ee9d9/afc7d43b-9f6f-4039-a896-6801bce38cb5"
-      (reference "C9") (unit 1) (value "100n") (footprint "Capacitor_SMD:C_0603_1608Metric")
+      (reference "C9") (unit 1) (value "1u") (footprint "Capacitor_SMD:C_0603_1608Metric")
     )
     (path "/dbae959f-bfa2-4953-9b3f-f4525f8ee9d9/70b2bcc7-30d0-4bb0-9597-39ba997d7a25"
@@
     )
     (path "/dbae959f-bfa2-4953-9b3f-f4525f8ee9d9/ea77193e-3f9c-4a16-9af4-44155de6e2bb"
-      (reference "C12") (unit 1) (value "100n") (footprint "Capacitor_SMD:C_0603_1608Metric")
+      (reference "C12") (unit 1) (value "1u") (footprint "Capacitor_SMD:C_0603_1608Metric")
     )
     (path "/dbae959f-bfa2-4953-9b3f-f4525f8ee9d9/a678b93c-ab66-4100-8ef3-b5ea0826667d"
-      (reference "C13") (unit 1) (value "100n") (footprint "Capacitor_SMD:C_0603_1608Metric")
+      (reference "C13") (unit 1) (value "1n") (footprint "Capacitor_SMD:C_0603_1608Metric")
     )
     (path "/dbae959f-bfa2-4953-9b3f-f4525f8ee9d9/f9bfe2eb-93b6-4c17-a75d-9f3361e33679"
-      (reference "C14") (unit 1) (value "100n") (footprint "Capacitor_SMD:C_0603_1608Metric")
+      (reference "C14") (unit 1) (value "1n") (footprint "Capacitor_SMD:C_0603_1608Metric")
     )
     (path "/fe9cb004-3747-4931-bcd5-b57852eb813d/1de3fe4d-6b8d-4612-8808-f29a2b0fe5ca"
@@
     )
     (path "/6785bf95-93a5-45b5-a636-e7169bb3f708/89aa4306-16cd-48dd-8c64-6203c30678e8"
-      (reference "L1") (unit 1) (value "L") (footprint "Inductor_SMD:L_0603_1608Metric")
+      (reference "L1") (unit 1) (value "600R") (footprint "Inductor_SMD:L_0603_1608Metric")
     )
     (path "/6785bf95-93a5-45b5-a636-e7169bb3f708/b1e5bead-33f6-48f8-893f-94df652ba665"
-      (reference "L2") (unit 1) (value "L") (footprint "Inductor_SMD:L_0603_1608Metric")
+      (reference "L2") (unit 1) (value "600R") (footprint "Inductor_SMD:L_0603_1608Metric")
     )
     (path "/dbae959f-bfa2-4953-9b3f-f4525f8ee9d9/89aa4306-16cd-48dd-8c64-6203c30678e8"
-      (reference "L3") (unit 1) (value "L") (footprint "Inductor_SMD:L_0603_1608Metric")
+      (reference "L3") (unit 1) (value "600R") (footprint "Inductor_SMD:L_0603_1608Metric")
     )
     (path "/dbae959f-bfa2-4953-9b3f-f4525f8ee9d9/b1e5bead-33f6-48f8-893f-94df652ba665"
-      (reference "L4") (unit 1) (value "L") (footprint "Inductor_SMD:L_0603_1608Metric")
+      (reference "L4") (unit 1) (value "600R") (footprint "Inductor_SMD:L_0603_1608Metric")
     )
     (path "/75a8b4cf-be6c-4d23-8740-2e62cd0245ef/df520658-f2c3-4297-b936-04f6ee7c468c"
@@
     )
     (path "/edaec270-515c-43bd-9198-429ba7237351"
-      (reference "R14") (unit 1) (value "10k") (footprint "Resistor_SMD:R_0603_1608Metric")
+      (reference "R14") (unit 1) (value "4k7") (footprint "Resistor_SMD:R_0603_1608Metric")
     )
     (path "/4b430f6f-d547-44b6-b4a5-c18ddad8f73b"
-      (reference "R15") (unit 1) (value "10k") (footprint "Resistor_SMD:R_0603_1608Metric")
+      (reference "R15") (unit 1) (value "4k7") (footprint "Resistor_SMD:R_0603_1608Metric")
     )
     (path "/6785bf95-93a5-45b5-a636-e7169bb3f708/bda8b78e-c7b4-4922-b8f7-5174c4ba8b8a"
@@
     )
     (path "/75a8b4cf-be6c-4d23-8740-2e62cd0245ef/38ea9190-7e44-4776-9df0-78109bd42804"
-      (reference "R43") (unit 1) (value "10k") (footprint "Resistor_SMD:R_0603_1608Metric")
+      (reference "R43") (unit 1) (value "110k") (footprint "Resistor_SMD:R_0603_1608Metric")
     )
     (path "/75a8b4cf-be6c-4d23-8740-2e62cd0245ef/e4f1bede-2e3e-4291-bdaa-a4b68bd8a25e"
-      (reference "R44") (unit 1) (value "10k") (footprint "Resistor_SMD:R_0603_1608Metric")
+      (reference "R44") (unit 1) (value "36k") (footprint "Resistor_SMD:R_0603_1608Metric")
     )
     (path "/75a8b4cf-be6c-4d23-8740-2e62cd0245ef/14eb34fb-fe53-42c2-b0d6-bb5cb7755bd1"
