File: KiCad/TFA9879.kicad_sch (KiCad schematic)
At the start: 20 parts, among them J4 Conn_01x02_Male, U2 TFA9879HN

Commit message: -First board version ready to order
Other:
- moved on the sheet: R16, R17
Changed lines of the file:
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@@
     (stroke (width 0) (type default) (color 0 0 0 0))
   )
-  (wire (pts (xy 60.96 116.84) (xy 85.09 116.84))
+  (wire (pts (xy 68.58 116.84) (xy 85.09 116.84))
     (stroke (width 0) (type default) (color 0 0 0 0))
   )
@@
     (stroke (width 0) (type default) (color 0 0 0 0))
   )
-  (wire (pts (xy 60.96 111.76) (xy 45.72 111.76))
+  (wire (pts (xy 53.34 111.76) (xy 45.72 111.76))
     (stroke (width 0) (type default) (color 0 0 0 0))
   )
@@
     (stroke (width 0) (type default) (color 0 0 0 0))
   )
-  (wire (pts (xy 68.58 111.76) (xy 74.93 111.76))
+  (wire (pts (xy 60.96 111.76) (xy 74.93 111.76))
     (stroke (width 0) (type default) (color 0 0 0 0))
   )
@@
     (stroke (width 0) (type default) (color 0 0 0 0))
   )
-  (wire (pts (xy 53.34 116.84) (xy 45.72 116.84))
+  (wire (pts (xy 60.96 116.84) (xy 45.72 116.84))
     (stroke (width 0) (type default) (color 0 0 0 0))
   )
@@
     (pin "2")
   )
-  (symbol (lib_id "Device:R") (at 57.15 116.84 90) (unit 1)
-    (in_bom yes) (on_board yes) (fields_autoplaced)
-    (property "Reference" "R16" (id 0) (at 57.15 110.49 90))
-    (property "Value" "110k" (id 1) (at 57.15 113.03 90))
-    (property "Footprint" "Resistor_SMD:R_0603_1608Metric" (id 2) (at 57.15 118.618 90)
-      (effects (font (size 1.27 1.27)) hide)
-    )
-    (property "Datasheet" "~" (id 3) (at 57.15 116.84 0)
-      (effects (font (size 1.27 1.27)) hide)
-    )
-    (pin "1")
-    (pin "2")
-  )
-  (symbol (lib_id "Device:R") (at 64.77 111.76 90) (unit 1)
-    (in_bom yes) (on_board yes) (fields_autoplaced)
-    (property "Reference" "R17" (id 0) (at 64.77 105.41 90))
-    (property "Value" "110k" (id 1) (at 64.77 107.95 90))
-    (property "Footprint" "Resistor_SMD:R_0603_1608Metric" (id 2) (at 64.77 113.538 90)
-      (effects (font (size 1.27 1.27)) hide)
-    )
-    (property "Datasheet" "~" (id 3) (at 64.77 111.76 0)
-      (effects (font (size 1.27 1.27)) hide)
-    )
+  (symbol (lib_id "Device:R") (at 64.77 116.84 90) (unit 1)
+    (in_bom yes) (on_board yes) (fields_autoplaced)
+    (property "Reference" "R16" (id 0) (at 64.77 110.49 90))
+    (property "Value" "110k" (id 1) (at 64.77 113.03 90))
+    (property "Footprint" "Resistor_SMD:R_0603_1608Metric" (id 2) (at 64.77 118.618 90)
+      (effects (font (size 1.27 1.27)) hide)
+    )
+    (property "Datasheet" "~" (id 3) (at 64.77 116.84 0)
+      (effects (font (size 1.27 1.27)) hide)
+    )
+    (pin "1")
+    (pin "2")
+  )
+  (symbol (lib_id "Device:R") (at 57.15 111.76 90) (unit 1)
+    (in_bom yes) (on_board yes) (fields_autoplaced)
+    (property "Reference" "R17" (id 0) (at 57.15 105.41 90))
+    (property "Value" "110k" (id 1) (at 57.15 107.95 90))
+    (property "Footprint" "Resistor_SMD:R_0603_1608Metric" (id 2) (at 57.15 113.538 90)
+      (effects (font (size 1.27 1.27)) hide)
+    )
+    (property "Datasheet" "~" (id 3) (at 57.15 111.76 0)
+      (effects (font (size 1.27 1.27)) hide)
+    )

Commit message: -updated schematic component values, updated schematic PDF -added simple bass and treble control for the TF9879 amp
Parts:
- C3, C6: value 100n -> 1u
- C7, C8: value 100n -> 1n
- L1, L2: value L -> 600R
Changed lines of the file:
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@@
     (in_bom yes) (on_board yes) (fields_autoplaced)
     (property "Reference" "L1" (id 0) (at 146.05 80.01 90))
-    (property "Value" "L" (id 1) (at 146.05 82.55 90))
+    (property "Value" "600R" (id 1) (at 146.05 82.55 90))
     (property "Footprint" "Inductor_SMD:L_0603_1608Metric" (id 2) (at 146.05 86.36 0)
       (effects (font (size 1.27 1.27)) hide)
@@
       (effects (font (size 1.27 1.27)) (justify left))
     )
-    (property "Value" "100n" (id 1) (at 158.75 116.8399 0)
+    (property "Value" "1n" (id 1) (at 158.75 116.8399 0)
       (effects (font (size 1.27 1.27)) (justify left))
     )
@@
       (effects (font (size 1.27 1.27)) (justify left))
     )
-    (property "Value" "100n" (id 1) (at 104.14 62.2299 0)
+    (property "Value" "1u" (id 1) (at 104.14 62.2299 0)
       (effects (font (size 1.27 1.27)) (justify left))
     )
@@
     (in_bom yes) (on_board yes) (fields_autoplaced)
     (property "Reference" "L2" (id 0) (at 146.05 90.17 90))
-    (property "Value" "L" (id 1) (at 146.05 92.71 90))
+    (property "Value" "600R" (id 1) (at 146.05 92.71 90))
     (property "Footprint" "Inductor_SMD:L_0603_1608Metric" (id 2) (at 146.05 96.52 0)
       (effects (font (size 1.27 1.27)) hide)
@@
       (effects (font (size 1.27 1.27)) (justify left))
     )
-    (property "Value" "100n" (id 1) (at 148.59 62.2299 0)
+    (property "Value" "1u" (id 1) (at 148.59 62.2299 0)
       (effects (font (size 1.27 1.27)) (justify left))
     )
@@
       (effects (font (size 1.27 1.27)) (justify left))
     )
-    (property "Value" "100n" (id 1) (at 171.45 116.8399 0)
-      (effects (font (size 1.27 1.27)) (justify left))
-    )
+    (property "Value" "1n" (id 1) (at 171.45 116.8399 0)
+      (effects (font (size 1.27 1.27)) (justify left))
+    )
